File: pizaid.sch (EAGLE design)
At the start: 44 parts, among them X1 S4B-ZR, X2 DCJACK-R

Commit message: ぐらんどきれいにした
Parts:
- R11: value (none) -> 10k
Changed lines of the file:
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@@
 <setting verticaltext="up"/>
 </settings>
-<grid distance="0.05" unitdist="inch" unit="inch" style="lines" multiple="1" display="no" altdistance="0.01" altunitdist="inch" altunit="inch"/>
+<grid distance="0.1" unitdist="inch" unit="inch" style="lines" multiple="1" display="no" altdistance="0.01" altunitdist="inch" altunit="inch"/>
 <layers>
 <layer number="1" name="Top" color="4" fill="1" visible="no" active="no"/>
@@
 <part name="R10" library="rcl" deviceset="R-US_" device="R0603" value="330"/>
 <part name="X1" library="con-jst" deviceset="?4B-ZR" device="S"/>
-<part name="R11" library="rcl" deviceset="R-US_" device="R0603"/>
+<part name="R11" library="rcl" deviceset="R-US_" device="R0603" value="10k"/>
 <part name="GND17" library="supply1" deviceset="GND" device=""/>
 <part name="U$8" library="pizaid" deviceset="B2P-VH" device=""/>

Commit message: modified board for stacking (ontheway)
Parts:
- removed S1: 10B-PH, con-jst:10B-PH
- removed U$14, U$15, U$9: B2P-VH, pizaid:B2P-VH
- removed X2: DCJACK-R, kamiki-dcjack:DCJACK-R
- added U$3: CON_14X2, pizaid:CON_14X2
- PCB1: device pizaid:RASPBERRY_PI_B+ -> RASPBERRY_PI_Bplus:RASPBERRY_PI_B+
- U$8: value B2P-VH -> CON_14X2; device pizaid:B2P-VH -> pizaid:CON_14X2
Connections:
- removed net 3V3@1: PCB1.3V3@1, S1G$2.1
- removed net GND@1: PCB1.GND@1
- removed net N$23: PCB1.GPIO27/GEN2, S1G$9.1
- new net B$1: PCB1.GPIO27/GEN2, U$8.P$2
- new net B1: PCB1.GPIO22/GEN3, U$8.P$4
- new net B10: PCB1.GPIO13, U$8.P$22
- new net B11: PCB1.GPIO19, U$8.P$24
- new net B12: PCB1.GPIO26, U$8.P$26
- new net B13: U$8.P$28
- new net B2: C10.1, PCB1.3V3@1, R14.2, R15.2, U$16.VCC, U$8.P$6
- new net B3: U$8.P$8
- new net B4: PCB1.GPIO9/MISO, U$8.P$10
- new net B5: PCB1.GPIO11/SCLK, U$8.P$12
- new net B6: U$8.P$14
- new net B7: U$8.P$16
- new net B8: PCB1.GPIO5, U$8.P$18
- new net B9: PCB1.GPIO6, U$8.P$20
- new net GND@3: PCB1.GND@1, PCB1.GND@2, PCB1.GND@3
- new net N$24: PCB1.!CE!/GPIO7, U$8.P$13
- new net N$25: PCB1.!CE0!/GPIO8, U$8.P$11
- new net N$26: PCB1.GEN/6GPIO25, U$8.P$9
- new net N$27: PCB1.GEN5/GPIO24, U$8.P$5
- new net N$28: PCB1.GEN4/GPIO23, U$8.P$3
- net 5V0@2: now also U$3.P$19, U$3.P$20, U$3.P$21, U$3.P$22, U$3.P$23; no longer C10.1, R14.2, R15.2, S1G$1.1, U$14G$1.1, U$16.VCC, U$9G$1.1
- net GND: now also U$3.P$14, U$3.P$15, U$3.P$16, U$3.P$17, U$3.P$18, U$3.P$24, U$3.P$25, U$3.P$26, U$3.P$27, U$3.P$28, U$3.P$5, U$3.P$6, U$3.P$7, U$3.P$8; no longer S1G$3.1, U$14G$2.1, U$15G$2.1, U$8G$2.1, U$9G$2.1, X2.2, X2.3
- net GND@4: now also PCB1.GND@5, PCB1.GND@6, PCB1.GND@7, U$8.P$1, U$8.P$17, U$8.P$21, U$8.P$7
- net JNET: now also U$3.P$10, U$3.P$11, U$3.P$12, U$3.P$13, U$3.P$9; no longer U$15G$1.1, U$8G$1.1
- net N$13: now also PCB1.GPIO20, U$8.P$25; no longer PCB1.TXD0/GPIO14, S1G$6.1
- net N$16: no longer S1G$5.1
- net N$20: no longer S1G$4.1
- net N$21: now also PCB1.GPIO16, U$8.P$23; no longer PCB1.RXD0/GPIO15, S1G$7.1
- net N$22: now also PCB1.GPIO12, U$8.P$19; no longer PCB1.GPIO18, S1G$8.1
- net N$9: now also PCB1.GPIO21, U$8.P$27; no longer PCB1.GPIO22/GEN3, S1G$10.1
- net VCC: now also U$3.P$1, U$3.P$2, U$3.P$3, U$3.P$4; no longer X2.1
Other:
- note removed: "+3.3V"
- note removed: "GND"
- note removed: "GPIOs"
- note removed: "SCL"
- note removed: "SDA"
- note removed: "Vcc"

Commit message: continuing placement.....................
Connections:
- net GND: now also U$3.P$1, U$3.P$2, U$3.P$3, U$3.P$4; no longer U$3.P$5, U$3.P$6, U$3.P$7, U$3.P$8
- net VCC: now also U$3.P$5, U$3.P$6, U$3.P$7, U$3.P$8; no longer U$3.P$1, U$3.P$2, U$3.P$3, U$3.P$4
Changed lines of the file:
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@@
 <setting verticaltext="up"/>
 </settings>
-<grid distance="0.05" unitdist="inch" unit="mm" style="lines" multiple="1" display="no" altdistance="0.01" altunitdist="inch" altunit="inch"/>
+<grid distance="0.05" unitdist="inch" unit="inch" style="lines" multiple="1" display="no" altdistance="0.01" altunitdist="inch" altunit="inch"/>
 <layers>
 <layer number="1" name="Top" color="4" fill="1" visible="no" active="no"/>
@@
 <instance part="P+1" gate="VCC" x="36.83" y="102.87"/>
 <instance part="U$2" gate="G$1" x="158.75" y="69.85" rot="R180"/>
-<instance part="P+2" gate="VCC" x="392.43" y="91.44"/>
+<instance part="P+2" gate="VCC" x="388.62" y="91.44"/>
 <instance part="U$4" gate="G$1" x="218.44" y="69.85" rot="R180"/>
 <instance part="U$5" gate="G$1" x="218.44" y="85.09" rot="R180"/>
@@
 <wire x1="420.37" y1="46.99" x2="422.91" y2="46.99" width="0.1524" layer="91"/>
 <junction x="422.91" y="46.99"/>
-<wire x1="422.91" y1="64.77" x2="422.91" y2="72.39" width="0.1524" layer="91"/>
+<wire x1="422.91" y1="64.77" x2="422.91" y2="77.47" width="0.1524" layer="91"/>
 <junction x="422.91" y="64.77"/>
-<pinref part="U$3" gate="G$1" pin="P$6"/>
-<wire x1="422.91" y1="72.39" x2="422.91" y2="74.93" width="0.1524" layer="91"/>
-<wire x1="422.91" y1="74.93" x2="420.37" y2="74.93" width="0.1524" layer="91"/>
-<pinref part="U$3" gate="G$1" pin="P$8"/>
-<wire x1="420.37" y1="72.39" x2="422.91" y2="72.39" width="0.1524" layer="91"/>
-<junction x="422.91" y="72.39"/>
+<pinref part="U$3" gate="G$1" pin="P$2"/>
+<wire x1="422.91" y1="77.47" x2="422.91" y2="80.01" width="0.1524" layer="91"/>
+<wire x1="422.91" y1="80.01" x2="420.37" y2="80.01" width="0.1524" layer="91"/>
+<pinref part="U$3" gate="G$1" pin="P$4"/>
+<wire x1="420.37" y1="77.47" x2="422.91" y2="77.47" width="0.1524" layer="91"/>
+<junction x="422.91" y="77.47"/>
 </segment>
 <segment>
@@
 <wire x1="394.97" y1="49.53" x2="392.43" y2="49.53" width="0.1524" layer="91"/>
 <junction x="392.43" y="49.53"/>
-<wire x1="392.43" y1="62.23" x2="392.43" y2="72.39" width="0.1524" layer="91"/>
+<wire x1="392.43" y1="62.23" x2="392.43" y2="77.47" width="0.1524" layer="91"/>
 <junction x="392.43" y="62.23"/>
-<pinref part="U$3" gate="G$1" pin="P$5"/>
-<wire x1="392.43" y1="72.39" x2="392.43" y2="74.93" width="0.1524" layer="91"/>
-<wire x1="392.43" y1="74.93" x2="394.97" y2="74.93" width="0.1524" layer="91"/>
-<pinref part="U$3" gate="G$1" pin="P$7"/>
-<wire x1="394.97" y1="72.39" x2="392.43" y2="72.39" width="0.1524" layer="91"/>
-<junction x="392.43" y="72.39"/>
+<pinref part="U$3" gate="G$1" pin="P$1"/>
+<wire x1="392.43" y1="77.47" x2="392.43" y2="80.01" width="0.1524" layer="91"/>
+<wire x1="392.43" y1="80.01" x2="394.97" y2="80.01" width="0.1524" layer="91"/>
+<pinref part="U$3" gate="G$1" pin="P$3"/>
+<wire x1="394.97" y1="77.47" x2="392.43" y2="77.47" width="0.1524" layer="91"/>
+<junction x="392.43" y="77.47"/>
 </segment>
 </net>
@@
 </segment>
 <segment>
-<pinref part="U$3" gate="G$1" pin="P$3"/>
+<pinref part="U$3" gate="G$1" pin="P$7"/>
 <pinref part="P+2" gate="VCC" pin="VCC"/>
-<wire x1="394.97" y1="77.47" x2="392.43" y2="77.47" width="0.1524" layer="91"/>
-<wire x1="392.43" y1="77.47" x2="392.43" y2="80.01" width="0.1524" layer="91"/>
-<pinref part="U$3" gate="G$1" pin="P$1"/>
-<wire x1="392.43" y1="80.01" x2="392.43" y2="86.36" width="0.1524" layer="91"/>
-<wire x1="392.43" y1="86.36" x2="392.43" y2="88.9" width="0.1524" layer="91"/>
-<wire x1="394.97" y1="80.01" x2="392.43" y2="80.01" width="0.1524" layer="91"/>
-<junction x="392.43" y="80.01"/>
-<wire x1="392.43" y1="86.36" x2="426.72" y2="86.36" width="0.1524" layer="91"/>
-<wire x1="426.72" y1="86.36" x2="426.72" y2="80.01" width="0.1524" layer="91"/>
-<junction x="392.43" y="86.36"/>
-<pinref part="U$3" gate="G$1" pin="P$4"/>
-<wire x1="426.72" y1="80.01" x2="426.72" y2="77.47" width="0.1524" layer="91"/>
-<wire x1="426.72" y1="77.47" x2="420.37" y2="77.47" width="0.1524" layer="91"/>
-<pinref part="U$3" gate="G$1" pin="P$2"/>
-<wire x1="420.37" y1="80.01" x2="426.72" y2="80.01" width="0.1524" layer="91"/>
-<junction x="426.72" y="80.01"/>
+<wire x1="394.97" y1="72.39" x2="388.62" y2="72.39" width="0.1524" layer="91"/>
+<wire x1="388.62" y1="72.39" x2="388.62" y2="74.93" width="0.1524" layer="91"/>
+<pinref part="U$3" gate="G$1" pin="P$5"/>
+<wire x1="388.62" y1="74.93" x2="388.62" y2="85.09" width="0.1524" layer="91"/>
+<wire x1="388.62" y1="85.09" x2="388.62" y2="88.9" width="0.1524" layer="91"/>
+<wire x1="394.97" y1="74.93" x2="388.62" y2="74.93" width="0.1524" layer="91"/>
+<junction x="388.62" y="74.93"/>
+<pinref part="U$3" gate="G$1" pin="P$8"/>
+<wire x1="420.37" y1="72.39" x2="426.72" y2="72.39" width="0.1524" layer="91"/>
+<wire x1="426.72" y1="72.39" x2="426.72" y2="74.93" width="0.1524" layer="91"/>
+<wire x1="426.72" y1="74.93" x2="426.72" y2="85.09" width="0.1524" layer="91"/>
+<wire x1="426.72" y1="85.09" x2="388.62" y2="85.09" width="0.1524" layer="91"/>
+<junction x="388.62" y="85.09"/>
+<pinref part="U$3" gate="G$1" pin="P$6"/>
+<wire x1="420.37" y1="74.93" x2="426.72" y2="74.93" width="0.1524" layer="91"/>
+<junction x="426.72" y="74.93"/>
 </segment>
 </net>

Commit message: updated second layer
Parts:
- removed X1: S4B-ZR, con-jst:S4B-ZR
- added R16: 10k, rcl:R-US_R0603
Connections:
- new net GIRD: C6.1, C8.1, R11.2, R16.2, U$4.K, U$5.K, U$6.VIN, U$7.VIN
- net GND: no longer X1-1.1
- net N$12: now also R16.1; no longer R11.1, U$6.ON/OFF, X1-4.1
- net N$8: now also R11.1, U$6.ON/OFF; no longer C6.1, C8.1, R11.2, U$4.K, U$5.K, U$6.VIN, U$7.VIN
Changed lines of the file:
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@@
 <part name="R9" library="rcl" deviceset="R-US_" device="R0603" value="1k"/>
 <part name="R10" library="rcl" deviceset="R-US_" device="R0603" value="330"/>
-<part name="X1" library="con-jst" deviceset="?4B-ZR" device="S"/>
 <part name="R11" library="rcl" deviceset="R-US_" device="R0603" value="10k"/>
-<part name="GND17" library="supply1" deviceset="GND" device=""/>
 <part name="U$10" library="pizaid" deviceset="B2P-VH" device=""/>
 <part name="GND18" library="supply1" deviceset="GND" device=""/>
@@
 <part name="GND20" library="supply1" deviceset="GND" device=""/>
 <part name="U$8" library="pizaid" deviceset="CON_14X2" device=""/>
+<part name="R16" library="rcl" deviceset="R-US_" device="R0603" value="10k"/>
 </parts>
 <sheets>
@@
 <instance part="R9" gate="G$1" x="335.28" y="-41.91"/>
 <instance part="R10" gate="G$1" x="349.25" y="-41.91"/>
-<instance part="X1" gate="-1" x="196.85" y="-44.45" rot="R180"/>
-<instance part="X1" gate="-2" x="196.85" y="-41.91" rot="R180"/>
-<instance part="X1" gate="-3" x="196.85" y="-39.37" rot="R180"/>
-<instance part="X1" gate="-4" x="196.85" y="-36.83" rot="R180"/>
 <instance part="R11" gate="G$1" x="238.76" y="57.15" rot="R90"/>
-<instance part="GND17" gate="1" x="205.74" y="-49.53"/>
 <instance part="U$10" gate="G$1" x="208.28" y="54.61"/>
 <instance part="U$10" gate="G$2" x="208.28" y="52.07"/>
@@
 <instance part="GND20" gate="1" x="422.91" y="41.91"/>
 <instance part="U$8" gate="G$1" x="345.44" y="-161.29"/>
+<instance part="R16" gate="G$1" x="228.6" y="57.15" rot="R90"/>
 </instances>
 <busses>
@@
 <pinref part="GND10" gate="1" pin="GND"/>
 <wire x1="340.36" y1="55.88" x2="340.36" y2="53.34" width="0.1524" layer="91"/>
-</segment>
-<segment>
-<pinref part="X1" gate="-1" pin="1"/>
-<pinref part="GND17" gate="1" pin="GND"/>
-<wire x1="201.93" y1="-44.45" x2="205.74" y2="-44.45" width="0.1524" layer="91"/>
-<wire x1="205.74" y1="-44.45" x2="205.74" y2="-46.99" width="0.1524" layer="91"/>
 </segment>
 <segment>
@@
 </segment>
 </net>
-<net name="N$8" class="0">
-<segment>
-<pinref part="U$5" gate="G$1" pin="K"/>
-<wire x1="223.52" y1="85.09" x2="232.41" y2="85.09" width="0.1524" layer="91"/>
-<wire x1="232.41" y1="85.09" x2="232.41" y2="69.85" width="0.1524" layer="91"/>
-<pinref part="U$4" gate="G$1" pin="K"/>
-<wire x1="232.41" y1="69.85" x2="223.52" y2="69.85" width="0.1524" layer="91"/>
-<pinref part="U$7" gate="G$1" pin="VIN"/>
-<wire x1="264.16" y1="-6.35" x2="256.54" y2="-6.35" width="0.1524" layer="91"/>
-<wire x1="256.54" y1="-6.35" x2="245.11" y2="-6.35" width="0.1524" layer="91"/>
-<wire x1="245.11" y1="-6.35" x2="245.11" y2="69.85" width="0.1524" layer="91"/>
-<wire x1="245.11" y1="69.85" x2="238.76" y2="69.85" width="0.1524" layer="91"/>
-<junction x="232.41" y="69.85"/>
-<pinref part="U$6" gate="G$1" pin="VIN"/>
-<wire x1="238.76" y1="69.85" x2="232.41" y2="69.85" width="0.1524" layer="91"/>
-<wire x1="264.16" y1="69.85" x2="256.54" y2="69.85" width="0.1524" layer="91"/>
-<junction x="245.11" y="69.85"/>
-<pinref part="C6" gate="G$1" pin="1"/>
-<wire x1="256.54" y1="69.85" x2="245.11" y2="69.85" width="0.1524" layer="91"/>
-<wire x1="256.54" y1="63.5" x2="256.54" y2="69.85" width="0.1524" layer="91"/>
-<junction x="256.54" y="69.85"/>
-<pinref part="C8" gate="G$1" pin="1"/>
-<wire x1="256.54" y1="-12.7" x2="256.54" y2="-6.35" width="0.1524" layer="91"/>
-<junction x="256.54" y="-6.35"/>
-<pinref part="R11" gate="G$1" pin="2"/>
-<wire x1="238.76" y1="62.23" x2="238.76" y2="69.85" width="0.1524" layer="91"/>
-<junction x="238.76" y="69.85"/>
-</segment>
-</net>
 <net name="N$14" class="0">
 <segment>
@@
 <pinref part="R8" gate="G$1" pin="1"/>
 <wire x1="340.36" y1="34.29" x2="344.17" y2="34.29" width="0.1524" layer="91"/>
-</segment>
-</net>
-<net name="N$12" class="0">
-<segment>
-<pinref part="U$6" gate="G$1" pin="ON/OFF"/>
-<pinref part="R11" gate="G$1" pin="1"/>
-<wire x1="264.16" y1="39.37" x2="238.76" y2="39.37" width="0.1524" layer="91"/>
-<wire x1="238.76" y1="39.37" x2="238.76" y2="52.07" width="0.1524" layer="91"/>
-<wire x1="238.76" y1="39.37" x2="238.76" y2="-36.83" width="0.1524" layer="91"/>
-<junction x="238.76" y="39.37"/>
-<pinref part="X1" gate="-4" pin="1"/>
-<wire x1="238.76" y1="-36.83" x2="201.93" y2="-36.83" width="0.1524" layer="91"/>
-<pinref part="U$7" gate="G$1" pin="ON/OFF"/>
-<wire x1="264.16" y1="-36.83" x2="238.76" y2="-36.83" width="0.1524" layer="91"/>
-<junction x="238.76" y="-36.83"/>
 </segment>
 </net>
@@
 </segment>
 </net>
+<net name="GIRD" class="0">
+<segment>
+<pinref part="U$5" gate="G$1" pin="K"/>
+<wire x1="223.52" y1="85.09" x2="232.41" y2="85.09" width="0.1524" layer="91"/>
+<wire x1="232.41" y1="85.09" x2="232.41" y2="69.85" width="0.1524" layer="91"/>
+<pinref part="U$4" gate="G$1" pin="K"/>
+<wire x1="232.41" y1="69.85" x2="228.6" y2="69.85" width="0.1524" layer="91"/>
+<pinref part="U$7" gate="G$1" pin="VIN"/>
+<wire x1="228.6" y1="69.85" x2="223.52" y2="69.85" width="0.1524" layer="91"/>
+<wire x1="264.16" y1="-6.35" x2="256.54" y2="-6.35" width="0.1524" layer="91"/>
+<wire x1="256.54" y1="-6.35" x2="245.11" y2="-6.35" width="0.1524" layer="91"/>
+<wire x1="245.11" y1="-6.35" x2="245.11" y2="69.85" width="0.1524" layer="91"/>
+<wire x1="245.11" y1="69.85" x2="238.76" y2="69.85" width="0.1524" layer="91"/>
+<junction x="232.41" y="69.85"/>
+<pinref part="U$6" gate="G$1" pin="VIN"/>
+<wire x1="238.76" y1="69.85" x2="232.41" y2="69.85" width="0.1524" layer="91"/>
+<wire x1="264.16" y1="69.85" x2="256.54" y2="69.85" width="0.1524" layer="91"/>
+<junction x="245.11" y="69.85"/>
+<pinref part="C6" gate="G$1" pin="1"/>
+<wire x1="256.54" y1="69.85" x2="245.11" y2="69.85" width="0.1524" layer="91"/>
+<wire x1="256.54" y1="63.5" x2="256.54" y2="69.85" width="0.1524" layer="91"/>
+<junction x="256.54" y="69.85"/>
+<pinref part="C8" gate="G$1" pin="1"/>
+<wire x1="256.54" y1="-12.7" x2="256.54" y2="-6.35" width="0.1524" layer="91"/>
+<junction x="256.54" y="-6.35"/>
+<pinref part="R11" gate="G$1" pin="2"/>
+<wire x1="238.76" y1="62.23" x2="238.76" y2="69.85" width="0.1524" layer="91"/>
+<junction x="238.76" y="69.85"/>
+<pinref part="R16" gate="G$1" pin="2"/>
+<wire x1="228.6" y1="62.23" x2="228.6" y2="69.85" width="0.1524" layer="91"/>
+<junction x="228.6" y="69.85"/>
+</segment>
+</net>
+<net name="N$8" class="0">
+<segment>
+<pinref part="R11" gate="G$1" pin="1"/>
+<pinref part="U$6" gate="G$1" pin="ON/OFF"/>
+<wire x1="264.16" y1="39.37" x2="238.76" y2="39.37" width="0.1524" layer="91"/>
+<wire x1="238.76" y1="39.37" x2="238.76" y2="52.07" width="0.1524" layer="91"/>
+</segment>
+</net>
+<net name="N$12" class="0">
+<segment>
+<pinref part="U$7" gate="G$1" pin="ON/OFF"/>
+<pinref part="R16" gate="G$1" pin="1"/>
+<wire x1="264.16" y1="-36.83" x2="228.6" y2="-36.83" width="0.1524" layer="91"/>
+<wire x1="228.6" y1="-36.83" x2="228.6" y2="52.07" width="0.1524" layer="91"/>
+</segment>
+</net>

Commit message: completed rev1
Parts:
- removed U$16: MCP3021, pizaid:MCP3021
- added U$9: MCP3425, pizaid:MCP3425
Connections:
- removed net GND@3: PCB1.GND@1, PCB1.GND@2, PCB1.GND@3
- removed net GND@4: PCB1.GND@4, PCB1.GND@5, PCB1.GND@6, PCB1.GND@7, PCB1.GND@8, U$8.P$1, U$8.P$17, U$8.P$21, U$8.P$7
- net B2: now also U$9.VCC; no longer U$16.VCC
- net GND: now also PCB1.GND@1, PCB1.GND@2, PCB1.GND@3, PCB1.GND@4, PCB1.GND@5, PCB1.GND@6, PCB1.GND@7, PCB1.GND@8, U$8.P$1, U$8.P$17, U$8.P$21, U$8.P$7, U$9.GND, U$9.VIN-; no longer U$16.GND
- net N$16: now also U$9.SCL; no longer U$16.SCL
- net N$19: now also U$9.VIN+; no longer U$16.AIN
- net N$20: now also U$9.SDA; no longer U$16.SDA
Other:
- moved on the sheet: C11
