File: pizaid.sch (EAGLE design)
At the start: 40 parts

Commit message: added gerber
Parts:
- R4: device rcl:R-US_0204/7 -> rcl:R-US_0207/10
Connections:
- removed net B7: U$8.P$16
- net 5V0@2: now also U$8.P$15, U$8.P$16
- net B2: now also PCB1.3V3@2
- net B3: now also PCB1.GPIO10/MOSI
Changed lines of the file:
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@@
 <setting verticaltext="up"/>
 </settings>
-<grid distance="0.1" unitdist="inch" unit="inch" style="lines" multiple="1" display="no" altdistance="0.01" altunitdist="inch" altunit="inch"/>
+<grid distance="0.05" unitdist="inch" unit="inch" style="lines" multiple="1" display="no" altdistance="0.01" altunitdist="inch" altunit="inch"/>
 <layers>
-<layer number="1" name="Top" color="4" fill="1" visible="no" active="no"/>
-<layer number="16" name="Bottom" color="1" fill="1" visible="no" active="no"/>
-<layer number="17" name="Pads" color="2" fill="1" visible="no" active="no"/>
-<layer number="18" name="Vias" color="2" fill="1" visible="no" active="no"/>
-<layer number="19" name="Unrouted" color="6" fill="1" visible="no" active="no"/>
-<layer number="20" name="Dimension" color="15" fill="1" visible="no" active="no"/>
-<layer number="21" name="tPlace" color="7" fill="1" visible="no" active="no"/>
-<layer number="22" name="bPlace" color="7" fill="1" visible="no" active="no"/>
-<layer number="23" name="tOrigins" color="15" fill="1" visible="no" active="no"/>
-<layer number="24" name="bOrigins" color="15" fill="1" visible="no" active="no"/>
-<layer number="25" name="tNames" color="7" fill="1" visible="no" active="no"/>
-<layer number="26" name="bNames" color="7" fill="1" visible="no" active="no"/>
-<layer number="27" name="tValues" color="7" fill="1" visible="no" active="no"/>
-<layer number="28" name="bValues" color="7" fill="1" visible="no" active="no"/>
+<layer number="1" name="Top" color="4" fill="1" visible="yes" active="no"/>
+<layer number="16" name="Bottom" color="1" fill="1" visible="yes" active="no"/>
+<layer number="17" name="Pads" color="2" fill="1" visible="yes" active="no"/>
+<layer number="18" name="Vias" color="2" fill="1" visible="yes" active="no"/>
+<layer number="19" name="Unrouted" color="6" fill="1" visible="yes" active="no"/>
+<layer number="20" name="Dimension" color="15" fill="1" visible="yes" active="no"/>
+<layer number="21" name="tPlace" color="7" fill="1" visible="yes" active="no"/>
+<layer number="22" name="bPlace" color="7" fill="1" visible="yes" active="no"/>
+<layer number="23" name="tOrigins" color="15" fill="1" visible="yes" active="no"/>
+<layer number="24" name="bOrigins" color="15" fill="1" visible="yes" active="no"/>
+<layer number="25" name="tNames" color="7" fill="1" visible="yes" active="no"/>
+<layer number="26" name="bNames" color="7" fill="1" visible="yes" active="no"/>
+<layer number="27" name="tValues" color="7" fill="1" visible="yes" active="no"/>
+<layer number="28" name="bValues" color="7" fill="1" visible="yes" active="no"/>
 <layer number="29" name="tStop" color="7" fill="3" visible="no" active="no"/>
 <layer number="30" name="bStop" color="7" fill="6" visible="no" active="no"/>
@@
 <layer number="35" name="tGlue" color="7" fill="4" visible="no" active="no"/>
 <layer number="36" name="bGlue" color="7" fill="5" visible="no" active="no"/>
-<layer number="37" name="tTest" color="7" fill="1" visible="no" active="no"/>
-<layer number="38" name="bTest" color="7" fill="1" visible="no" active="no"/>
+<layer number="37" name="tTest" color="7" fill="1" visible="yes" active="no"/>
+<layer number="38" name="bTest" color="7" fill="1" visible="yes" active="no"/>
 <layer number="39" name="tKeepout" color="4" fill="11" visible="no" active="no"/>
 <layer number="40" name="bKeepout" color="1" fill="11" visible="no" active="no"/>
@@
 <layer number="44" name="Drills" color="7" fill="1" visible="no" active="no"/>
 <layer number="45" name="Holes" color="7" fill="1" visible="no" active="no"/>
-<layer number="46" name="Milling" color="3" fill="1" visible="no" active="no"/>
-<layer number="47" name="Measures" color="7" fill="1" visible="no" active="no"/>
-<layer number="48" name="Document" color="7" fill="1" visible="no" active="no"/>
-<layer number="49" name="Reference" color="7" fill="1" visible="no" active="no"/>
-<layer number="51" name="tDocu" color="7" fill="1" visible="no" active="no"/>
-<layer number="52" name="bDocu" color="7" fill="1" visible="no" active="no"/>
+<layer number="46" name="Milling" color="3" fill="1" visible="yes" active="no"/>
+<layer number="47" name="Measures" color="7" fill="1" visible="yes" active="no"/>
+<layer number="48" name="Document" color="7" fill="1" visible="yes" active="no"/>
+<layer number="49" name="Reference" color="7" fill="1" visible="yes" active="no"/>
+<layer number="51" name="tDocu" color="7" fill="1" visible="yes" active="no"/>
+<layer number="52" name="bDocu" color="7" fill="1" visible="yes" active="no"/>
 <layer number="91" name="Nets" color="2" fill="1" visible="yes" active="yes"/>
 <layer number="92" name="Busses" color="1" fill="1" visible="yes" active="yes"/>
@@
 <part name="R2" library="rcl" deviceset="R-US_" device="R0603" value="10k"/>
 <part name="R3" library="rcl" deviceset="R-US_" device="R0603" value="2.2k"/>
-<part name="R4" library="rcl" deviceset="R-US_" device="0204/7" value="0.2"/>
+<part name="R4" library="rcl" deviceset="R-US_" device="0207/10" value="0.2"/>
 <part name="R5" library="rcl" deviceset="R-US_" device="R0603" value="24"/>
 <part name="R6" library="rcl" deviceset="R-US_" device="R0603" value="1k"/>
@@
 <wire x1="426.72" y1="54.61" x2="426.72" y2="57.15" width="0.1524" layer="91"/>
 <junction x="426.72" y="57.15"/>
+<wire x1="328.93" y1="-130.81" x2="328.93" y2="-137.16" width="0.1524" layer="91"/>
+<junction x="328.93" y="-130.81"/>
+<pinref part="U$8" gate="G$1" pin="P$15"/>
+<wire x1="328.93" y1="-137.16" x2="328.93" y2="-163.83" width="0.1524" layer="91"/>
+<wire x1="328.93" y1="-163.83" x2="332.74" y2="-163.83" width="0.1524" layer="91"/>
+<pinref part="U$8" gate="G$1" pin="P$16"/>
+<wire x1="358.14" y1="-163.83" x2="361.95" y2="-163.83" width="0.1524" layer="91"/>
+<wire x1="361.95" y1="-163.83" x2="361.95" y2="-137.16" width="0.1524" layer="91"/>
+<wire x1="361.95" y1="-137.16" x2="328.93" y2="-137.16" width="0.1524" layer="91"/>
+<junction x="328.93" y="-137.16"/>
 </segment>
 </net>
@@
 <net name="B2" class="0">
 <segment>
-<wire x1="266.7" y1="-151.13" x2="254" y2="-151.13" width="0.1524" layer="91"/>
 <pinref part="PCB1" gate="G$1" pin="3V3@1"/>
 <wire x1="254" y1="-151.13" x2="248.92" y2="-151.13" width="0.1524" layer="91"/>
@@
 <junction x="260.35" y="-130.81"/>
 <wire x1="254" y1="-130.81" x2="254" y2="-151.13" width="0.1524" layer="91"/>
+<pinref part="U$9" gate="G$1" pin="VCC"/>
+<pinref part="PCB1" gate="G$1" pin="3V3@2"/>
+<wire x1="265.43" y1="-151.13" x2="254" y2="-151.13" width="0.1524" layer="91"/>
 <junction x="254" y="-151.13"/>
-<pinref part="U$9" gate="G$1" pin="VCC"/>
 </segment>
 <segment>
@@
 <net name="B3" class="0">
 <segment>
-<wire x1="266.7" y1="-153.67" x2="248.92" y2="-153.67" width="0.1524" layer="91"/>
-</segment>
-<segment>
 <pinref part="U$8" gate="G$1" pin="P$8"/>
 <wire x1="358.14" y1="-153.67" x2="372.11" y2="-153.67" width="0.1524" layer="91"/>
+</segment>
+<segment>
+<pinref part="PCB1" gate="G$1" pin="GPIO10/MOSI"/>
+<wire x1="265.43" y1="-153.67" x2="248.92" y2="-153.67" width="0.1524" layer="91"/>
 </segment>
 </net>
@@
 </segment>
 </net>
-<net name="B7" class="0">
-<segment>
-<pinref part="U$8" gate="G$1" pin="P$16"/>
-<wire x1="358.14" y1="-163.83" x2="372.11" y2="-163.83" width="0.1524" layer="91"/>
-</segment>
-</net>

Commit message: modified battery board to output 12V
Parts:
- removed C8: 22u25V, rcl:C-EUC3225
- removed C9: 22u16V, rcl:C-EUC3225
- removed R10: 330, rcl:R-US_R0603
- removed R11, R16: 10k, rcl:R-US_R0603
- removed R9: 1k, rcl:R-US_R0603
- removed U$7: OKL-T/6, pizaid:OKL-T/6
- added U$11: SELECT_PAD, pizaid:SELECT_PAD
- added X1: DCJACK-MJ179P-R, kamiki-dcjack:DCJACK-MJ179P-R
Connections:
- removed net JNET: C7.1, U$3.P$10, U$3.P$11, U$3.P$12, U$3.P$13, U$3.P$9, U$6.SENSE, U$6.VOUT
- removed net N$12: R16.1, U$7.ON/OFF
- removed net N$14: R9.1, U$7.TRIM
- removed net N$15: R10.1, R9.2
- removed net N$8: R11.1, U$6.ON/OFF
- new net N$30: U$11.P$2, U$3.P$10, U$3.P$11, U$3.P$12, U$3.P$13, U$3.P$19, U$3.P$20, U$3.P$21, U$3.P$22, U$3.P$23, U$3.P$9
- net 5V0@2: now also C7.1, U$11.P$3, U$6.SENSE, U$6.VOUT; no longer C9.1, U$3.P$19, U$3.P$20, U$3.P$21, U$3.P$22, U$3.P$23, U$7.SENSE, U$7.VOUT
- net GIRD: now also U$11.P$1; no longer C8.1, R11.2, R16.2, U$7.VIN
- net GND: now also U$6.ON/OFF, X1.2, X1.3; no longer C8.2, C9.2, R10.2, U$7.GND@1, U$7.GND@2
- net VCC: now also X1.1
Other:
- moved on the sheet: C10, C11, PCB1, R12, R13, R14, R15
