File: pizaid.sch (EAGLE design)
At the start: 35 parts, among them X1 DCJACK-MJ179P-R

Commit message: add default output jumper to 5V
Parts:
- R4: device rcl:R-US_0207/10 -> rcl:R-US_0207/15
Connections:
- removed net N$30: U$11.P$2, U$3.P$10, U$3.P$11, U$3.P$12, U$3.P$13, U$3.P$19, U$3.P$20, U$3.P$21, U$3.P$22, U$3.P$23, U$3.P$9
- net 5V0@2: now also U$11.P$2, U$3.P$10, U$3.P$11, U$3.P$12, U$3.P$13, U$3.P$19, U$3.P$20, U$3.P$21, U$3.P$22, U$3.P$23, U$3.P$9

Commit message: add AVR and bug fix
Connections:
- removed net N$28: PCB1.GEN4/GPIO23, U$8.P$3
- net B$1: no longer U$8.P$2
- net N$16: now also U$8.P$2
- net N$20: now also U$8.P$3
Changed lines of the file:
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@@
 <grid distance="0.05" unitdist="inch" unit="inch" style="lines" multiple="1" display="no" altdistance="0.01" altunitdist="inch" altunit="inch"/>
 <layers>
-<layer number="1" name="Top" color="4" fill="1" visible="yes" active="no"/>
-<layer number="16" name="Bottom" color="1" fill="1" visible="yes" active="no"/>
-<layer number="17" name="Pads" color="2" fill="1" visible="yes" active="no"/>
-<layer number="18" name="Vias" color="2" fill="1" visible="yes" active="no"/>
-<layer number="19" name="Unrouted" color="6" fill="1" visible="yes" active="no"/>
-<layer number="20" name="Dimension" color="15" fill="1" visible="yes" active="no"/>
-<layer number="21" name="tPlace" color="7" fill="1" visible="yes" active="no"/>
-<layer number="22" name="bPlace" color="7" fill="1" visible="yes" active="no"/>
-<layer number="23" name="tOrigins" color="15" fill="1" visible="yes" active="no"/>
-<layer number="24" name="bOrigins" color="15" fill="1" visible="yes" active="no"/>
-<layer number="25" name="tNames" color="7" fill="1" visible="yes" active="no"/>
-<layer number="26" name="bNames" color="7" fill="1" visible="yes" active="no"/>
-<layer number="27" name="tValues" color="7" fill="1" visible="yes" active="no"/>
-<layer number="28" name="bValues" color="7" fill="1" visible="yes" active="no"/>
+<layer number="1" name="Top" color="4" fill="1" visible="no" active="no"/>
+<layer number="16" name="Bottom" color="1" fill="1" visible="no" active="no"/>
+<layer number="17" name="Pads" color="2" fill="1" visible="no" active="no"/>
+<layer number="18" name="Vias" color="2" fill="1" visible="no" active="no"/>
+<layer number="19" name="Unrouted" color="6" fill="1" visible="no" active="no"/>
+<layer number="20" name="Dimension" color="15" fill="1" visible="no" active="no"/>
+<layer number="21" name="tPlace" color="7" fill="1" visible="no" active="no"/>
+<layer number="22" name="bPlace" color="7" fill="1" visible="no" active="no"/>
+<layer number="23" name="tOrigins" color="15" fill="1" visible="no" active="no"/>
+<layer number="24" name="bOrigins" color="15" fill="1" visible="no" active="no"/>
+<layer number="25" name="tNames" color="7" fill="1" visible="no" active="no"/>
+<layer number="26" name="bNames" color="7" fill="1" visible="no" active="no"/>
+<layer number="27" name="tValues" color="7" fill="1" visible="no" active="no"/>
+<layer number="28" name="bValues" color="7" fill="1" visible="no" active="no"/>
 <layer number="29" name="tStop" color="7" fill="3" visible="no" active="no"/>
 <layer number="30" name="bStop" color="7" fill="6" visible="no" active="no"/>
@@
 <layer number="35" name="tGlue" color="7" fill="4" visible="no" active="no"/>
 <layer number="36" name="bGlue" color="7" fill="5" visible="no" active="no"/>
-<layer number="37" name="tTest" color="7" fill="1" visible="yes" active="no"/>
-<layer number="38" name="bTest" color="7" fill="1" visible="yes" active="no"/>
+<layer number="37" name="tTest" color="7" fill="1" visible="no" active="no"/>
+<layer number="38" name="bTest" color="7" fill="1" visible="no" active="no"/>
 <layer number="39" name="tKeepout" color="4" fill="11" visible="no" active="no"/>
 <layer number="40" name="bKeepout" color="1" fill="11" visible="no" active="no"/>
@@
 <layer number="44" name="Drills" color="7" fill="1" visible="no" active="no"/>
 <layer number="45" name="Holes" color="7" fill="1" visible="no" active="no"/>
-<layer number="46" name="Milling" color="3" fill="1" visible="yes" active="no"/>
-<layer number="47" name="Measures" color="7" fill="1" visible="yes" active="no"/>
-<layer number="48" name="Document" color="7" fill="1" visible="yes" active="no"/>
-<layer number="49" name="Reference" color="7" fill="1" visible="yes" active="no"/>
-<layer number="51" name="tDocu" color="7" fill="1" visible="yes" active="no"/>
-<layer number="52" name="bDocu" color="7" fill="1" visible="yes" active="no"/>
+<layer number="46" name="Milling" color="3" fill="1" visible="no" active="no"/>
+<layer number="47" name="Measures" color="7" fill="1" visible="no" active="no"/>
+<layer number="48" name="Document" color="7" fill="1" visible="no" active="no"/>
+<layer number="49" name="Reference" color="7" fill="1" visible="no" active="no"/>
+<layer number="51" name="tDocu" color="7" fill="1" visible="no" active="no"/>
+<layer number="52" name="bDocu" color="7" fill="1" visible="no" active="no"/>
 <layer number="91" name="Nets" color="2" fill="1" visible="yes" active="yes"/>
 <layer number="92" name="Busses" color="1" fill="1" visible="yes" active="yes"/>
@@
 <pinref part="R15" gate="G$1" pin="1"/>
 <wire x1="242.57" y1="-45.72" x2="242.57" y2="-33.02" width="0.1524" layer="91"/>
-<wire x1="242.57" y1="-33.02" x2="242.57" y2="-11.43" width="0.1524" layer="91"/>
+<wire x1="242.57" y1="-33.02" x2="242.57" y2="-17.78" width="0.1524" layer="91"/>
+<wire x1="242.57" y1="-17.78" x2="242.57" y2="-11.43" width="0.1524" layer="91"/>
 <wire x1="227.33" y1="-45.72" x2="242.57" y2="-45.72" width="0.1524" layer="91"/>
 <wire x1="265.43" y1="-33.02" x2="242.57" y2="-33.02" width="0.1524" layer="91"/>
@@
 <pinref part="PCB1" gate="G$1" pin="GPIO3/SCL1"/>
 <pinref part="U$9" gate="G$1" pin="SCL"/>
+<pinref part="U$8" gate="G$1" pin="P$2"/>
+<wire x1="358.14" y1="-43.18" x2="365.76" y2="-43.18" width="0.1524" layer="91"/>
+<wire x1="365.76" y1="-43.18" x2="365.76" y2="-17.78" width="0.1524" layer="91"/>
+<wire x1="365.76" y1="-17.78" x2="242.57" y2="-17.78" width="0.1524" layer="91"/>
+<junction x="242.57" y="-17.78"/>
 </segment>
 </net>
@@
 <pinref part="R14" gate="G$1" pin="1"/>
 <wire x1="233.68" y1="-35.56" x2="233.68" y2="-30.48" width="0.1524" layer="91"/>
-<wire x1="233.68" y1="-30.48" x2="233.68" y2="-11.43" width="0.1524" layer="91"/>
+<wire x1="233.68" y1="-30.48" x2="233.68" y2="-20.32" width="0.1524" layer="91"/>
+<wire x1="233.68" y1="-20.32" x2="233.68" y2="-11.43" width="0.1524" layer="91"/>
 <wire x1="233.68" y1="-35.56" x2="227.33" y2="-35.56" width="0.1524" layer="91"/>
 <wire x1="265.43" y1="-30.48" x2="233.68" y2="-30.48" width="0.1524" layer="91"/>
@@
 <pinref part="PCB1" gate="G$1" pin="GPIO2/SDA1"/>
 <pinref part="U$9" gate="G$1" pin="SDA"/>
+<pinref part="U$8" gate="G$1" pin="P$3"/>
+<wire x1="332.74" y1="-45.72" x2="325.12" y2="-45.72" width="0.1524" layer="91"/>
+<wire x1="325.12" y1="-45.72" x2="325.12" y2="-20.32" width="0.1524" layer="91"/>
+<wire x1="325.12" y1="-20.32" x2="233.68" y2="-20.32" width="0.1524" layer="91"/>
+<junction x="233.68" y="-20.32"/>
 </segment>
 </net>
@@
 </segment>
 </net>
-<net name="N$28" class="0">
-<segment>
-<pinref part="U$8" gate="G$1" pin="P$3"/>
-<pinref part="PCB1" gate="G$1" pin="GEN4/GPIO23"/>
-<wire x1="332.74" y1="-45.72" x2="313.69" y2="-45.72" width="0.1524" layer="91"/>
-</segment>
-</net>
 <net name="B$1" class="0">
 <segment>
@@
 <wire x1="265.43" y1="-43.18" x2="248.92" y2="-43.18" width="0.1524" layer="91"/>
 </segment>
-<segment>
-<pinref part="U$8" gate="G$1" pin="P$2"/>
-<wire x1="358.14" y1="-43.18" x2="372.11" y2="-43.18" width="0.1524" layer="91"/>
-</segment>
-</net>
+</net>
